File: cc2652rb_v3.sch (EAGLE design)
At the start: 38 parts, among them IC2 CP2102, J3 CORTEX_DEBUG_SMD, J5 TYPE-C-31-M-12, Q3 SI2323DS, U1 E72-2G4M05S1F, U2 3.3V

Commit message: Add files via upload
Parts:
- C13: value (none) -> 220uF
Connections:
- net DIO_3: now also J2.15; no longer J1.19
- net GND: now also J1.19; no longer J2.15
Changed lines of the file:
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@@
 <part name="GND1" library="supply1" library_urn="urn:adsk.eagle:library:371" deviceset="GND" device=""/>
 <part name="GND2" library="supply1" library_urn="urn:adsk.eagle:library:371" deviceset="GND" device=""/>
-<part name="C13" library="Capacitor" library_urn="urn:adsk.eagle:library:16290819" deviceset="C" device="TANTALUM-2917(7343-METRIC)" package3d_urn="urn:adsk.eagle:package:16290891/2" technology="_"/>
+<part name="C13" library="Capacitor" library_urn="urn:adsk.eagle:library:16290819" deviceset="C" device="TANTALUM-2917(7343-METRIC)" package3d_urn="urn:adsk.eagle:package:16290891/2" technology="_" value="220uF"/>
 <part name="C14" library="SparkFun-Capacitors" deviceset="10UF" device="-0603-6.3V-20%" package3d_urn="urn:adsk.eagle:package:37414/1" value="10uF"/>
 <part name="C15" library="SparkFun-Capacitors" deviceset="1.0UF" device="-0603-16V-10%" package3d_urn="urn:adsk.eagle:package:37414/1" value="1.0uF"/>
@@
 <attribute name="VALUE" x="215.9" y="12.7" size="1.778" layer="96"/>
 </instance>
-<instance part="GND9" gate="1" x="271.78" y="83.82" smashed="yes" rot="R90">
-<attribute name="VALUE" x="274.32" y="81.28" size="1.778" layer="96" rot="R90"/>
+<instance part="GND9" gate="1" x="271.78" y="81.28" smashed="yes" rot="R90">
+<attribute name="VALUE" x="274.32" y="78.74" size="1.778" layer="96" rot="R90"/>
 </instance>
 <instance part="GND10" gate="1" x="358.14" y="35.56" smashed="yes">
@@
 </segment>
 <segment>
-<pinref part="J1" gate="G$1" pin="19"/>
-<wire x1="228.6" y1="93.98" x2="236.22" y2="93.98" width="0.1524" layer="91"/>
-<label x="228.6" y="93.98" size="1.778" layer="95"/>
-</segment>
-<segment>
 <pinref part="IC2" gate="G$1" pin="RXD"/>
 <wire x1="78.74" y1="30.48" x2="88.9" y2="30.48" width="0.1524" layer="91"/>
 <label x="81.28" y="30.48" size="1.778" layer="95"/>
+</segment>
+<segment>
+<pinref part="J2" gate="G$1" pin="15"/>
+<wire x1="261.62" y1="83.82" x2="269.24" y2="83.82" width="0.1524" layer="91"/>
+<label x="261.62" y="83.82" size="1.778" layer="95"/>
 </segment>
 </net>
@@
 </segment>
 <segment>
-<pinref part="J2" gate="G$1" pin="15"/>
-<wire x1="261.62" y1="83.82" x2="269.24" y2="83.82" width="0.1524" layer="91"/>
 <pinref part="GND9" gate="1" pin="GND"/>
 <pinref part="J2" gate="G$1" pin="14"/>
 <wire x1="261.62" y1="81.28" x2="269.24" y2="81.28" width="0.1524" layer="91"/>
-<wire x1="269.24" y1="81.28" x2="269.24" y2="83.82" width="0.1524" layer="91"/>
-<junction x="269.24" y="83.82"/>
 </segment>
 <segment>
@@
 <pinref part="GND16" gate="1" pin="GND"/>
 </segment>
-</net>
+<segment>
+<pinref part="J1" gate="G$1" pin="19"/>
+<wire x1="228.6" y1="93.98" x2="236.22" y2="93.98" width="0.1524" layer="91"/>
+<label x="231.14" y="93.98" size="1.778" layer="95"/>
+</segment>
+</net>

Commit message: Add files via upload
Parts:
- removed C14: 10uF, SparkFun-Capacitors:10UF-0603-6.3V-20%
- removed C15: 1.0uF, SparkFun-Capacitors:1.0UF-0603-16V-10%
- removed C16: 0.1uF, SparkFun-Capacitors:0.1UF-0603-25V-(+80/-20%)
- removed C17: 100pF, SparkFun-Capacitors:100PF-0603-50V-5%
- added J4: (no value), SparkFun-Connectors:QWIIC_CONNECTORJS-1MM
Connections:
- net DIO_4: now also J4.SCL
- net DIO_5: now also J4.SDA
- net GND: now also J4.GND; no longer C14.2, C15.2, C16.2, C17.2
- net VCC: now also J4.VCC; no longer C14.1, C15.1, C16.1, C17.1
Changed lines of the file:
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@@
 <part name="GND2" library="supply1" library_urn="urn:adsk.eagle:library:371" deviceset="GND" device=""/>
 <part name="C13" library="Capacitor" library_urn="urn:adsk.eagle:library:16290819" deviceset="C" device="TANTALUM-2917(7343-METRIC)" package3d_urn="urn:adsk.eagle:package:16290891/2" technology="_" value="220uF"/>
-<part name="C14" library="SparkFun-Capacitors" deviceset="10UF" device="-0603-6.3V-20%" package3d_urn="urn:adsk.eagle:package:37414/1" value="10uF"/>
-<part name="C15" library="SparkFun-Capacitors" deviceset="1.0UF" device="-0603-16V-10%" package3d_urn="urn:adsk.eagle:package:37414/1" value="1.0uF"/>
-<part name="C16" library="SparkFun-Capacitors" deviceset="0.1UF" device="-0603-25V-(+80/-20%)" package3d_urn="urn:adsk.eagle:package:37414/1" value="0.1uF"/>
-<part name="C17" library="SparkFun-Capacitors" deviceset="100PF" device="-0603-50V-5%" package3d_urn="urn:adsk.eagle:package:37414/1" value="100pF"/>
 <part name="GND3" library="supply1" library_urn="urn:adsk.eagle:library:371" deviceset="GND" device=""/>
 <part name="BTN1" library="SparkFun-Switches" library_urn="urn:adsk.eagle:library:535" deviceset="MOMENTARY-SWITCH-SPST-2" device="-SMD-4.6X2.8MM" package3d_urn="urn:adsk.eagle:package:40176/1"/>
@@
 <part name="J3" library="SparkFun-Connectors" deviceset="CORTEX_DEBUG" device="_SMD" package3d_urn="urn:adsk.eagle:package:38289/1"/>
 <part name="GND16" library="supply1" library_urn="urn:adsk.eagle:library:371" deviceset="GND" device=""/>
+<part name="J4" library="SparkFun-Connectors" deviceset="QWIIC_CONNECTOR" device="JS-1MM" package3d_urn="urn:adsk.eagle:package:38096/1"/>
 </parts>
 <sheets>
@@
 <attribute name="VALUE" x="305.816" y="72.009" size="1.778" layer="96" font="vector"/>
 </instance>
-<instance part="C14" gate="G$1" x="312.42" y="73.66" smashed="yes">
-<attribute name="NAME" x="313.944" y="76.581" size="1.778" layer="95" font="vector"/>
-<attribute name="VALUE" x="313.944" y="71.501" size="1.778" layer="96" font="vector"/>
-</instance>
-<instance part="C15" gate="G$1" x="320.04" y="73.66" smashed="yes">
-<attribute name="NAME" x="321.564" y="76.581" size="1.778" layer="95" font="vector"/>
-<attribute name="VALUE" x="321.564" y="71.501" size="1.778" layer="96" font="vector"/>
-</instance>
-<instance part="C16" gate="G$1" x="327.66" y="73.66" smashed="yes">
-<attribute name="NAME" x="329.184" y="76.581" size="1.778" layer="95" font="vector"/>
-<attribute name="VALUE" x="329.184" y="71.501" size="1.778" layer="96" font="vector"/>
-</instance>
-<instance part="C17" gate="G$1" x="335.28" y="73.66" smashed="yes">
-<attribute name="NAME" x="336.804" y="76.581" size="1.778" layer="95" font="vector"/>
-<attribute name="VALUE" x="336.804" y="71.501" size="1.778" layer="96" font="vector"/>
-</instance>
-<instance part="GND3" gate="1" x="335.28" y="60.96" smashed="yes">
-<attribute name="VALUE" x="332.74" y="58.42" size="1.778" layer="96"/>
+<instance part="GND3" gate="1" x="304.8" y="63.5" smashed="yes">
+<attribute name="VALUE" x="302.26" y="60.96" size="1.778" layer="96"/>
 </instance>
 <instance part="BTN1" gate="G$1" x="251.46" y="22.86" smashed="yes">
@@
 <instance part="GND16" gate="1" x="104.14" y="50.8" smashed="yes">
 <attribute name="VALUE" x="101.6" y="48.26" size="1.778" layer="96"/>
+</instance>
+<instance part="J4" gate="J1" x="320.04" y="76.2" smashed="yes">
+<attribute name="VALUE" x="314.96" y="70.866" size="1.778" layer="96" font="vector" align="top-left"/>
+<attribute name="NAME" x="314.96" y="84.074" size="1.778" layer="95" font="vector"/>
 </instance>
 </instances>
@@
 <label x="228.6" y="88.9" size="1.778" layer="95"/>
 </segment>
+<segment>
+<pinref part="J4" gate="J1" pin="SDA"/>
+<wire x1="327.66" y1="78.74" x2="337.82" y2="78.74" width="0.1524" layer="91"/>
+<label x="330.2" y="78.74" size="1.778" layer="95"/>
+</segment>
 </net>
 <net name="DIO_4" class="0">
@@
 <label x="228.6" y="91.44" size="1.778" layer="95"/>
 </segment>
+<segment>
+<pinref part="J4" gate="J1" pin="SCL"/>
+<wire x1="327.66" y1="81.28" x2="337.82" y2="81.28" width="0.1524" layer="91"/>
+<label x="330.2" y="81.28" size="1.778" layer="95"/>
+</segment>
 </net>
 <net name="DIO_3" class="0">
@@
 </segment>
 <segment>
-<pinref part="C17" gate="G$1" pin="1"/>
-<wire x1="312.42" y1="83.82" x2="320.04" y2="83.82" width="0.1524" layer="91"/>
-<wire x1="320.04" y1="83.82" x2="327.66" y2="83.82" width="0.1524" layer="91"/>
-<wire x1="327.66" y1="83.82" x2="335.28" y2="83.82" width="0.1524" layer="91"/>
-<wire x1="335.28" y1="83.82" x2="335.28" y2="78.74" width="0.1524" layer="91"/>
-<pinref part="C14" gate="G$1" pin="1"/>
-<wire x1="312.42" y1="78.74" x2="312.42" y2="83.82" width="0.1524" layer="91"/>
-<pinref part="C15" gate="G$1" pin="1"/>
-<wire x1="320.04" y1="78.74" x2="320.04" y2="83.82" width="0.1524" layer="91"/>
-<junction x="320.04" y="83.82"/>
-<pinref part="C16" gate="G$1" pin="1"/>
-<wire x1="327.66" y1="78.74" x2="327.66" y2="83.82" width="0.1524" layer="91"/>
-<junction x="327.66" y="83.82"/>
-<wire x1="335.28" y1="83.82" x2="345.44" y2="83.82" width="0.1524" layer="91"/>
-<junction x="335.28" y="83.82"/>
-<label x="340.36" y="83.82" size="1.778" layer="95"/>
+<label x="304.8" y="78.74" size="1.778" layer="95" rot="R90"/>
 <pinref part="C13" gate="G$1" pin="1"/>
 <wire x1="304.8" y1="78.74" x2="304.8" y2="83.82" width="0.1524" layer="91"/>
-<wire x1="304.8" y1="83.82" x2="312.42" y2="83.82" width="0.1524" layer="91"/>
-<junction x="312.42" y="83.82"/>
 </segment>
 <segment>
@@
 <label x="104.14" y="63.5" size="1.778" layer="95"/>
 </segment>
+<segment>
+<pinref part="J4" gate="J1" pin="VCC"/>
+<wire x1="327.66" y1="76.2" x2="337.82" y2="76.2" width="0.1524" layer="91"/>
+<label x="332.74" y="76.2" size="1.778" layer="95"/>
+</segment>
 </net>
 <net name="DIO_30" class="0">
@@
 <wire x1="228.6" y1="48.26" x2="236.22" y2="48.26" width="0.1524" layer="91"/>
 <label x="228.6" y="48.26" size="1.778" layer="95"/>
-</segment>
-<segment>
-<pinref part="C13" gate="G$1" pin="2"/>
-<wire x1="304.8" y1="71.12" x2="304.8" y2="66.04" width="0.1524" layer="91"/>
-<pinref part="C17" gate="G$1" pin="2"/>
-<wire x1="304.8" y1="66.04" x2="312.42" y2="66.04" width="0.1524" layer="91"/>
-<wire x1="312.42" y1="66.04" x2="320.04" y2="66.04" width="0.1524" layer="91"/>
-<wire x1="320.04" y1="66.04" x2="327.66" y2="66.04" width="0.1524" layer="91"/>
-<wire x1="327.66" y1="66.04" x2="335.28" y2="66.04" width="0.1524" layer="91"/>
-<wire x1="335.28" y1="66.04" x2="335.28" y2="71.12" width="0.1524" layer="91"/>
-<pinref part="C14" gate="G$1" pin="2"/>
-<wire x1="312.42" y1="71.12" x2="312.42" y2="66.04" width="0.1524" layer="91"/>
-<junction x="312.42" y="66.04"/>
-<pinref part="C15" gate="G$1" pin="2"/>
-<wire x1="320.04" y1="71.12" x2="320.04" y2="66.04" width="0.1524" layer="91"/>
-<junction x="320.04" y="66.04"/>
-<pinref part="C16" gate="G$1" pin="2"/>
-<wire x1="327.66" y1="71.12" x2="327.66" y2="66.04" width="0.1524" layer="91"/>
-<junction x="327.66" y="66.04"/>
-<wire x1="335.28" y1="63.5" x2="335.28" y2="66.04" width="0.1524" layer="91"/>
-<junction x="335.28" y="66.04"/>
-<pinref part="GND3" gate="1" pin="GND"/>
 </segment>
 <segment>
@@
 <label x="231.14" y="93.98" size="1.778" layer="95"/>
 </segment>
-</net>
+<segment>
+<pinref part="C13" gate="G$1" pin="2"/>
+<wire x1="304.8" y1="71.12" x2="304.8" y2="66.04" width="0.1524" layer="91"/>
+<pinref part="GND3" gate="1" pin="GND"/>
+</segment>
+<segment>
+<pinref part="J4" gate="J1" pin="GND"/>
+<wire x1="327.66" y1="73.66" x2="337.82" y2="73.66" width="0.1524" layer="91"/>
+<label x="332.74" y="73.66" size="1.778" layer="95"/>
+</segment>
+</net>
