File: 3.1/cc2652rb_v3.1.brd (EAGLE design)
At the start: 25.3 x 57.3 mm, 32 parts, among them J3 CORTEX_DEBUG_SMD, J5 TYPE-C-31-M-12, Q3 SI2323DS, U1 E72-2G4M05S1F, U2 3.3V, U3 CH340E_MSOP10

Commit message: Add files via upload
Parts:
- removed C14: 10uF, SparkFun-Capacitors:0603
- removed C15: 1.0uF, SparkFun-Capacitors:0603
- removed C16: 0.1uF, SparkFun-Capacitors:0603
- removed C17: 100pF, SparkFun-Capacitors:0603
- added C4: 0.1uF, SparkFun-Capacitors:0603
- added I2C: (no value), SparkFun-Connectors:1X04_1MM_RA
- added Y1: Q22FA12800150, ok-xtal-osc-dev:XTAL-4P-2016
- moved R4 0.70 mm to (9.00, 11.4)
Connections:
- new net X48M_N: U1.34, Y1.3
- new net X48M_P: U1.35, Y1.1
- net +5V: now also C4.2, U3.10
- net DIO_4: now also I2C.4
- net DIO_5: now also I2C.3
- net GND: now also C4.1, I2C.1, Y1.2, Y1.4; no longer C14.2, C15.2, C16.2, C17.2
- net VCC: now also I2C.2; no longer C14.1, C15.1, C16.1, C17.1
Routing:
- net VCC: track 78.9 -> 94.1 mm
- net +5V: track 32.2 -> 38.8 mm
- net DIO_5: track 3.63 -> 8.76 mm, vias 0 -> 1
- net X48M_P: track 0.00 -> 5.12 mm, vias 0 -> 1
- net GND: track 13.3 -> 16.5 mm, vias 95 -> 90
- net DIO_4: track 3.63 -> 6.58 mm, vias 0 -> 1
- net X48M_N: track 0.00 -> 2.62 mm, vias 0 -> 1

Commit message: Add files via upload
Parts:
- turned C4 to 90 degrees
Connections:
- net +5V: no longer C4.2, U3.10, U3.7
- net LDO: now also C4.2, U3.10, U3.7
Routing:
- net LDO: track 17.3 -> 46.3 mm, vias 2 -> 4
- net +5V: track 38.8 -> 27.4 mm, vias 4 -> 3
Changed lines of the file:
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@@
 <drawing>
 <settings>
-<setting alwaysvectorfont="no"/>
+<setting alwaysvectorfont="yes"/>
 <setting verticaltext="up"/>
 </settings>
@@
 <attribute name="PRICE" value="None" x="12.3" y="14.2" size="1.778" layer="27" rot="R180" display="off"/>
 </element>
-<element name="C4" library="SparkFun-Capacitors" package="0603" package3d_urn="urn:adsk.eagle:package:37414/1" value="0.1uF" x="7.5" y="10.8" smashed="yes" rot="R270">
-<attribute name="NAME" x="7.462" y="12.6" size="0.8128" layer="25" font="vector" ratio="20" align="bottom-center"/>
-<attribute name="PROD_ID" value="CAP-00810" x="7.5" y="10.8" size="1.778" layer="27" rot="R270" display="off"/>
+<element name="C4" library="SparkFun-Capacitors" package="0603" package3d_urn="urn:adsk.eagle:package:37414/1" value="0.1uF" x="7.5" y="10.8" smashed="yes" rot="R90">
+<attribute name="NAME" x="7.538" y="13.3" size="0.8128" layer="25" font="vector" ratio="20" rot="R180" align="bottom-center"/>
+<attribute name="PROD_ID" value="CAP-00810" x="7.5" y="10.8" size="1.778" layer="27" rot="R90" display="off"/>
 </element>
 <element name="Y1" library="ok-xtal-osc-dev" package="XTAL-4P-2016" value="Q22FA12800150" x="17.4" y="41.4" smashed="yes" rot="MR180">
@@
 <via x="14.7" y="20.3" extent="1-16" drill="0.3"/>
 <via x="5.4" y="20.8" extent="1-16" drill="0.3"/>
-<via x="16.2" y="14.7" extent="1-16" drill="0.3"/>
 <via x="10.1" y="17.2" extent="1-16" drill="0.3"/>
 <via x="19.6" y="27.7" extent="1-16" drill="0.3"/>
@@
 <via x="17.6" y="36.9" extent="1-16" drill="0.3"/>
 <via x="19.3" y="34.3" extent="1-16" drill="0.3"/>
+<via x="16.7" y="14.3" extent="1-16" drill="0.3"/>
 </signal>
 <signal name="RESET">
@@
 <wire x1="15.1161625" y1="9.5" x2="15.7" y2="9.5" width="0.508" layer="1"/>
 <via x="15.7" y="9.5" extent="1-16" drill="0.3"/>
-<wire x1="12.5" y1="12.5" x2="12.3" y2="12.3" width="0.508" layer="16"/>
 <via x="12.3" y="12.3" extent="1-16" drill="0.3"/>
 <wire x1="13.355" y1="11.76" x2="12.44" y2="11.76" width="0.2" layer="1"/>
 <wire x1="12.44" y1="11.76" x2="12.3" y2="11.9" width="0.2" layer="1"/>
 <wire x1="12.3" y1="11.9" x2="12.3" y2="12.3" width="0.2" layer="1"/>
-<wire x1="12.3" y1="12.3" x2="14.5" y2="12.3" width="0.508" layer="16"/>
-<wire x1="15.7" y1="11.1" x2="15.7" y2="9.5" width="0.508" layer="16"/>
-<wire x1="14.5" y1="12.3" x2="15.7" y2="11.1" width="0.508" layer="16"/>
-<wire x1="12.5" y1="15.4" x2="15.1" y2="15.4" width="0.508" layer="16"/>
-<wire x1="15.1" y1="15.4" x2="15.8" y2="16.1" width="0.508" layer="16"/>
-<wire x1="15.8" y1="16.1" x2="15.8" y2="16.9" width="0.508" layer="16"/>
-<contactref element="U3" pad="7"/>
-<via x="12.5" y="15.4" extent="1-16" drill="0.3"/>
-<wire x1="12.5" y1="15.4" x2="12.5" y2="12.5" width="0.508" layer="16"/>
-<wire x1="10.05" y1="14.7" x2="11.6" y2="14.7" width="0.254" layer="1"/>
-<wire x1="11.6" y1="14.7" x2="11.8" y2="14.7" width="0.254" layer="1"/>
-<wire x1="11.8" y1="14.7" x2="12.5" y2="15.4" width="0.254" layer="1"/>
-<contactref element="U3" pad="10"/>
-<contactref element="C4" pad="2"/>
-<wire x1="9.85" y1="7.995" x2="9.85" y2="8.95" width="0.254" layer="1"/>
-<wire x1="9.85" y1="8.95" x2="8.85" y2="9.95" width="0.254" layer="1"/>
-<wire x1="8.85" y1="9.95" x2="7.5" y2="9.95" width="0.254" layer="1"/>
-<wire x1="10.05" y1="13.2" x2="11.2" y2="13.2" width="0.2" layer="1"/>
-<wire x1="11.6" y1="13.6" x2="11.6" y2="14.7" width="0.2" layer="1"/>
-<wire x1="11.2" y1="13.2" x2="11.6" y2="13.6" width="0.2" layer="1"/>
+<wire x1="15.8" y1="16.9" x2="15.8" y2="12.3" width="0.508" layer="16"/>
+<wire x1="15.8" y1="12.3" x2="15.8" y2="9.6" width="0.508" layer="16"/>
+<wire x1="15.8" y1="9.6" x2="15.7" y2="9.5" width="0.508" layer="16"/>
+<wire x1="12.3" y1="12.3" x2="15.8" y2="12.3" width="0.508" layer="16"/>
 </signal>
 <signal name="N$2">
@@
 <wire x1="19" y1="15.3" x2="18.6" y2="15.7" width="0.508" layer="1"/>
 <wire x1="18.6" y1="15.7" x2="18.6" y2="15.9" width="0.508" layer="1"/>
+<contactref element="U3" pad="7"/>
+<contactref element="U3" pad="10"/>
+<contactref element="C4" pad="2"/>
+<wire x1="10.05" y1="13.2" x2="11.2" y2="13.2" width="0.2" layer="1"/>
+<wire x1="11.5" y1="13.5" x2="11.5" y2="14.5" width="0.2" layer="1"/>
+<wire x1="11.5" y1="14.5" x2="11.3" y2="14.7" width="0.2" layer="1"/>
+<wire x1="11.3" y1="14.7" x2="10.05" y2="14.7" width="0.2" layer="1"/>
+<wire x1="11.2" y1="13.2" x2="11.5" y2="13.5" width="0.2" layer="1"/>
+<wire x1="10.05" y1="14.7" x2="8.9" y2="14.7" width="0.2" layer="1"/>
+<wire x1="8.9" y1="14.7" x2="8.7" y2="14.9" width="0.2" layer="1"/>
+<via x="8.7" y="14.9" extent="1-16" drill="0.3"/>
+<wire x1="18.6" y1="15.9" x2="18.6" y2="10.9" width="0.3048" layer="16"/>
+<wire x1="16.542" y1="8.842" x2="9.758" y2="8.842" width="0.3048" layer="16"/>
+<wire x1="9.758" y1="8.842" x2="8.7" y2="9.9" width="0.3048" layer="16"/>
+<wire x1="8.7" y1="9.9" x2="8.7" y2="12.8" width="0.3048" layer="16"/>
+<wire x1="8.7" y1="12.8" x2="8.7" y2="14.9" width="0.3048" layer="16"/>
+<wire x1="18.6" y1="10.9" x2="16.542" y2="8.842" width="0.3048" layer="16"/>
+<wire x1="7.5" y1="11.65" x2="7.5" y2="12.7" width="0.254" layer="1"/>
+<wire x1="7.5" y1="12.7" x2="7.6" y2="12.8" width="0.254" layer="1"/>
+<via x="7.6" y="12.8" extent="1-16" drill="0.3"/>
+<wire x1="7.6" y1="12.8" x2="8.7" y2="12.8" width="0.3048" layer="16"/>
 </signal>
 <signal name="CC2">

Commit message: Add files via upload
Parts:
- removed C3: 0.1uF, SparkFun-Capacitors:0603
- removed R1: 100k, RC0402FR-073M6L:RESC1005X40N
- moved BTN2 4.53 mm to (18.2, 26.9), turned to 180 degrees
- moved Y1 0.20 mm to (17.6, 41.4), turned to 270 degrees
Connections:
- net GND: no longer C3.2
- net RESET: no longer C3.1, R1.2
- net VCC: no longer R1.1
Routing:
- net RESET: track 79.7 -> 76.2 mm
- net DIO_14: track 43.2 -> 46.1 mm
- net X48M_P: track 5.12 -> 2.59 mm
- net X48M_N: track 2.62 -> 4.68 mm
- net GND: track 16.5 -> 15.2 mm, vias 90 -> 86

Commit message: Add files via upload
Parts:
- removed Y1: Q22FA12800150, ok-xtal-osc-dev:XTAL-4P-2016
- added C20, C22: 7p, discretes-dev:CAPC1005X40N
- added Y2: Q22FA12800150, ok-xtal-osc-dev:XTAL-4P-2016
- R11: value 10k -> 100k
- moved BTN2 0.30 mm to (18.2, 26.6)
Connections:
- removed net X48M_N: U1.34, Y1.3
- removed net X48M_P: U1.35, Y1.1
- new net N$1: C20.1, U1.35, Y2.1
- new net N$4: C22.2, U1.34, Y2.3
- net GND: now also Y2.2, Y2.4; no longer Y1.2, Y1.4
Routing:
- net N$1: track 0.00 -> 6.00 mm, vias 0 -> 1
- net X48M_N: track 4.68 -> 0.00 mm, vias 1 -> 0
- net N$4: track 0.00 -> 3.89 mm, vias 0 -> 1
- net X48M_P: track 2.59 -> 0.00 mm, vias 1 -> 0
- net GND: track 15.2 -> 16.6 mm, vias 86 -> 89
Other:
- outline, holes or cut-outs redrawn
