File: 3.1/cc2652rb_v3.1.sch (EAGLE design)
At the start: 32 parts, among them J3 CORTEX_DEBUG_SMD, J5 TYPE-C-31-M-12, Q3 SI2323DS, U1 E72-2G4M05S1F, U2 3.3V, U3 CH340E_MSOP10

Commit message: Add files via upload
Parts:
- removed C14: 10uF, SparkFun-Capacitors:10UF-0603-6.3V-20%
- removed C15: 1.0uF, SparkFun-Capacitors:1.0UF-0603-16V-10%
- removed C16: 0.1uF, SparkFun-Capacitors:0.1UF-0603-25V-(+80/-20%)
- removed C17: 100pF, SparkFun-Capacitors:100PF-0603-50V-5%
- added C4: 0.1uF, SparkFun-Capacitors:0.1UF-0603-25V-(+80/-20%)
- added I2C: (no value), SparkFun-Connectors:QWIIC_CONNECTORJS-1MM
- added Y1: Q22FA12800150, ok-xtal-osc-dev:48.000MHZ_CX2016DB48000C0FPLC1
Connections:
- new net X48M_N: U1.X48M-N, Y1.3
- new net X48M_P: U1.X48N-P, Y1.1
- net +5V: now also C4.2, U3.V3
- net DIO_4: now also I2C.SCL
- net DIO_5: now also I2C.SDA
- net GND: now also C4.1, I2C.GND, Y1.2, Y1.4; no longer C14.2, C15.2, C16.2, C17.2
- net VCC: now also I2C.VCC; no longer C14.1, C15.1, C16.1, C17.1
Other:
- moved on the sheet: BT1, C13, D1, D2, D5, J1, J2, Q3, R11, R3, R5

Commit message: Add files via upload
Connections:
- net +5V: no longer C4.2, U3.V3, U3.VCC
- net LDO: now also C4.2, U3.V3, U3.VCC
Other:
- moved on the sheet: C4
Changed lines of the file:
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@@
 <part name="U3" library="CH340E" deviceset="CH340E" device="_MSOP10"/>
 <part name="GND20" library="supply1" library_urn="urn:adsk.eagle:library:371" deviceset="GND" device=""/>
-<part name="P+7" library="supply1" library_urn="urn:adsk.eagle:library:371" deviceset="+5V" device=""/>
 <part name="C4" library="SparkFun-Capacitors" deviceset="0.1UF" device="-0603-25V-(+80/-20%)" package3d_urn="urn:adsk.eagle:package:37414/1" value="0.1uF"/>
 <part name="GND11" library="supply1" library_urn="urn:adsk.eagle:library:371" deviceset="GND" device=""/>
@@
 <wire x1="210.82" y1="96.52" x2="220.98" y2="86.36" width="0.3048" layer="94"/>
 <wire x1="210.82" y1="86.36" x2="220.98" y2="96.52" width="0.3048" layer="94"/>
+<wire x1="53.34" y1="58.42" x2="86.36" y2="33.02" width="0.508" layer="94"/>
+<wire x1="53.34" y1="33.02" x2="83.82" y2="58.42" width="0.508" layer="94"/>
 </plain>
 <instances>
@@
 <attribute name="VALUE" x="0" y="25.4" size="1.778" layer="96"/>
 </instance>
-<instance part="P+7" gate="1" x="2.54" y="58.42" smashed="yes">
-<attribute name="VALUE" x="0" y="53.34" size="1.778" layer="96" rot="R90"/>
-</instance>
-<instance part="C4" gate="G$1" x="-5.08" y="48.26" smashed="yes" rot="R90">
-<attribute name="NAME" x="-8.001" y="49.784" size="1.778" layer="95" font="vector" rot="R90"/>
-<attribute name="VALUE" x="-2.921" y="49.784" size="1.778" layer="96" font="vector" rot="R90"/>
-</instance>
-<instance part="GND11" gate="1" x="-15.24" y="48.26" smashed="yes" rot="R270">
-<attribute name="VALUE" x="-17.78" y="50.8" size="1.778" layer="96" rot="R270"/>
+<instance part="C4" gate="G$1" x="-5.08" y="50.8" smashed="yes" rot="R90">
+<attribute name="NAME" x="-8.001" y="52.324" size="1.778" layer="95" font="vector" rot="R90"/>
+<attribute name="VALUE" x="-2.921" y="52.324" size="1.778" layer="96" font="vector" rot="R90"/>
+</instance>
+<instance part="GND11" gate="1" x="-15.24" y="50.8" smashed="yes" rot="R270">
+<attribute name="VALUE" x="-17.78" y="53.34" size="1.778" layer="96" rot="R270"/>
 </instance>
 <instance part="Y1" gate="G$1" x="215.9" y="91.44" smashed="yes">
@@
 <segment>
 <pinref part="C4" gate="G$1" pin="1"/>
-<wire x1="-10.16" y1="48.26" x2="-12.7" y2="48.26" width="0.1524" layer="91"/>
+<wire x1="-10.16" y1="50.8" x2="-12.7" y2="50.8" width="0.1524" layer="91"/>
 <pinref part="GND11" gate="1" pin="GND"/>
 </segment>
@@
 <wire x1="50.8" y1="104.14" x2="50.8" y2="106.68" width="0.1524" layer="91"/>
 <pinref part="P+5" gate="1" pin="+5V"/>
-</segment>
-<segment>
-<pinref part="U3" gate="U1" pin="VCC"/>
-<wire x1="5.08" y1="50.8" x2="2.54" y2="50.8" width="0.1524" layer="91"/>
-<wire x1="2.54" y1="50.8" x2="2.54" y2="55.88" width="0.1524" layer="91"/>
-<pinref part="P+7" gate="1" pin="+5V"/>
-<pinref part="U3" gate="U1" pin="V3"/>
-<wire x1="5.08" y1="48.26" x2="2.54" y2="48.26" width="0.1524" layer="91"/>
-<wire x1="2.54" y1="48.26" x2="2.54" y2="50.8" width="0.1524" layer="91"/>
-<junction x="2.54" y="50.8"/>
-<pinref part="C4" gate="G$1" pin="2"/>
-<wire x1="2.54" y1="48.26" x2="-2.54" y2="48.26" width="0.1524" layer="91"/>
-<junction x="2.54" y="48.26"/>
 </segment>
 </net>
@@
 <label x="358.14" y="91.44" size="1.778" layer="95"/>
 </segment>
-</net>
+<segment>
+<pinref part="U3" gate="U1" pin="VCC"/>
+<wire x1="5.08" y1="50.8" x2="2.54" y2="50.8" width="0.1524" layer="91"/>
+<pinref part="U3" gate="U1" pin="V3"/>
+<wire x1="5.08" y1="48.26" x2="2.54" y2="48.26" width="0.1524" layer="91"/>
+<wire x1="2.54" y1="48.26" x2="2.54" y2="50.8" width="0.1524" layer="91"/>
+<junction x="2.54" y="50.8"/>
+<pinref part="C4" gate="G$1" pin="2"/>
+<wire x1="2.54" y1="50.8" x2="-2.54" y2="50.8" width="0.1524" layer="91"/>
+<wire x1="2.54" y1="50.8" x2="2.54" y2="58.42" width="0.1524" layer="91"/>
+<label x="2.54" y="53.34" size="1.778" layer="95" rot="R90"/>
+</segment>
+</net>

Commit message: Add files via upload
Parts:
- removed C3: 0.1uF, SparkFun-Capacitors:0.1UF-0603-25V-(+80/-20%)
- removed R1: 100k, RC0402FR-073M6L:RC0402FR-073M6L
Connections:
- net GND: no longer C3.2
- net RESET: no longer C3.1, R1.2
- net VCC: no longer R1.1
Changed lines of the file:
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@@
 <part name="C2" library="SparkFun-Capacitors" library_urn="urn:adsk.eagle:library:510" deviceset="10UF" device="-0603-6.3V-20%" package3d_urn="urn:adsk.eagle:package:37414/1" value="10uF"/>
 <part name="P+1" library="supply1" library_urn="urn:adsk.eagle:library:371" deviceset="+5V" device=""/>
-<part name="R1" library="RC0402FR-073M6L" deviceset="RC0402FR-073M6L" device="" value="100k"/>
-<part name="C3" library="SparkFun-Capacitors" deviceset="0.1UF" device="-0603-25V-(+80/-20%)" package3d_urn="urn:adsk.eagle:package:37414/1" value="0.1uF"/>
-<part name="GND8" library="supply1" library_urn="urn:adsk.eagle:library:371" deviceset="GND" device=""/>
 <part name="GND9" library="supply1" library_urn="urn:adsk.eagle:library:371" deviceset="GND" device=""/>
 <part name="GND10" library="supply1" library_urn="urn:adsk.eagle:library:371" deviceset="GND" device=""/>
@@
 <attribute name="VALUE" x="99.06" y="99.06" size="1.778" layer="96" rot="R90"/>
 </instance>
-<instance part="R1" gate="G$1" x="220.98" y="40.64" smashed="yes" rot="R180">
-<attribute name="NAME" x="220.98" y="39.116" size="1.778" layer="95" font="vector" rot="R180" align="bottom-center"/>
-</instance>
-<instance part="C3" gate="G$1" x="218.44" y="22.86" smashed="yes">
-<attribute name="NAME" x="219.964" y="25.781" size="1.778" layer="95" font="vector"/>
-<attribute name="VALUE" x="219.964" y="20.701" size="1.778" layer="96" font="vector"/>
-</instance>
-<instance part="GND8" gate="1" x="218.44" y="15.24" smashed="yes">
-<attribute name="VALUE" x="215.9" y="12.7" size="1.778" layer="96"/>
-</instance>
 <instance part="GND9" gate="1" x="292.1" y="81.28" smashed="yes" rot="R90">
 <attribute name="VALUE" x="294.64" y="78.74" size="1.778" layer="96" rot="R90"/>
@@
 <net name="RESET" class="0">
 <segment>
-<pinref part="C3" gate="G$1" pin="1"/>
-<wire x1="208.28" y1="30.48" x2="218.44" y2="30.48" width="0.1524" layer="91"/>
-<wire x1="218.44" y1="30.48" x2="218.44" y2="27.94" width="0.1524" layer="91"/>
 <pinref part="U1" gate="G$1" pin="RESET_N"/>
-<pinref part="R1" gate="G$1" pin="2"/>
-<wire x1="200.66" y1="40.64" x2="208.28" y2="40.64" width="0.1524" layer="91"/>
-<wire x1="208.28" y1="40.64" x2="210.82" y2="40.64" width="0.1524" layer="91"/>
-<wire x1="208.28" y1="30.48" x2="208.28" y2="40.64" width="0.1524" layer="91"/>
-<junction x="208.28" y="40.64"/>
+<wire x1="200.66" y1="40.64" x2="210.82" y2="40.64" width="0.1524" layer="91"/>
 <label x="203.2" y="40.64" size="1.778" layer="95"/>
 </segment>
@@
 </segment>
 <segment>
-<pinref part="R1" gate="G$1" pin="1"/>
-<wire x1="231.14" y1="40.64" x2="236.22" y2="40.64" width="0.1524" layer="91"/>
-<label x="231.14" y="40.64" size="1.778" layer="95"/>
-</segment>
-<segment>
 <pinref part="D5" gate="G$1" pin="C"/>
 <wire x1="373.38" y1="83.82" x2="375.92" y2="83.82" width="0.1524" layer="91"/>
@@
 </segment>
 <segment>
-<pinref part="C3" gate="G$1" pin="2"/>
-<wire x1="218.44" y1="20.32" x2="218.44" y2="17.78" width="0.1524" layer="91"/>
-<pinref part="GND8" gate="1" pin="GND"/>
-</segment>
-<segment>

Commit message: Add files via upload
Parts:
- removed Y1: Q22FA12800150, ok-xtal-osc-dev:48.000MHZ_CX2016DB48000C0FPLC1
- added C20, C22: 7p, discretes-dev:CAP0402
- added Y2: Q22FA12800150, ok-xtal-osc-dev:48.000MHZ_CX2016DB48000C0FPLC1
- R11: value 10k -> 100k
Connections:
- removed net X48M_N: U1.X48M-N, Y1.3
- removed net X48M_P: U1.X48N-P, Y1.1
- new net N$1: C20.1, U1.X48N-P, Y2.1
- new net N$4: C22.2, U1.X48M-N, Y2.3
- net GND: now also Y2.2, Y2.4; no longer Y1.2, Y1.4
Changed lines of the file:
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@@
 <part name="Q3" library="SI2323DS" deviceset="SI2323DS" device=""/>
 <part name="D5" library="diode" library_urn="urn:adsk.eagle:library:210" deviceset="BAT60J" device="" package3d_urn="urn:adsk.eagle:package:43461/1"/>
-<part name="R11" library="RC0402FR-073M6L" deviceset="RC0402FR-073M6L" device="" value="10k"/>
+<part name="R11" library="RC0402FR-073M6L" deviceset="RC0402FR-073M6L" device="" value="100k"/>
 <part name="BT1" library="Battery Holder_2" deviceset="79527141" device="" package3d_urn="urn:adsk.eagle:package:12584890/3"/>
 <part name="GND4" library="supply1" library_urn="urn:adsk.eagle:library:371" deviceset="GND" device=""/>
@@
 <part name="C4" library="SparkFun-Capacitors" deviceset="0.1UF" device="-0603-25V-(+80/-20%)" package3d_urn="urn:adsk.eagle:package:37414/1" value="0.1uF"/>
 <part name="GND11" library="supply1" library_urn="urn:adsk.eagle:library:371" deviceset="GND" device=""/>
-<part name="Y1" library="ok-xtal-osc-dev" deviceset="48.000MHZ_CX2016DB48000C0FPLC1" device="" value="Q22FA12800150"/>
+<part name="I2C" library="SparkFun-Connectors" deviceset="QWIIC_CONNECTOR" device="JS-1MM" package3d_urn="urn:adsk.eagle:package:38096/1"/>
+<part name="Y2" library="ok-xtal-osc-dev" deviceset="48.000MHZ_CX2016DB48000C0FPLC1" device="" value="Q22FA12800150"/>
+<part name="C20" library="discretes-dev" deviceset="CAP0402" device="" value="7p"/>
+<part name="C22" library="discretes-dev" deviceset="CAP0402" device="" value="7p"/>
 <part name="GND19" library="supply1" library_urn="urn:adsk.eagle:library:371" deviceset="GND" device=""/>
 <part name="GND21" library="supply1" library_urn="urn:adsk.eagle:library:371" deviceset="GND" device=""/>
-<part name="I2C" library="SparkFun-Connectors" deviceset="QWIIC_CONNECTOR" device="JS-1MM" package3d_urn="urn:adsk.eagle:package:38096/1"/>
+<part name="GND23" library="supply1" library_urn="urn:adsk.eagle:library:371" deviceset="GND" device=""/>
 </parts>
 <sheets>
 <sheet>
 <plain>
-<wire x1="210.82" y1="96.52" x2="220.98" y2="86.36" width="0.3048" layer="94"/>
-<wire x1="210.82" y1="86.36" x2="220.98" y2="96.52" width="0.3048" layer="94"/>
+<wire x1="215.9" y1="99.06" x2="226.06" y2="88.9" width="0.3048" layer="94"/>
+<wire x1="215.9" y1="88.9" x2="226.06" y2="99.06" width="0.3048" layer="94"/>
 <wire x1="53.34" y1="58.42" x2="86.36" y2="33.02" width="0.508" layer="94"/>
 <wire x1="53.34" y1="33.02" x2="83.82" y2="58.42" width="0.508" layer="94"/>
@@
 <attribute name="VALUE" x="-17.78" y="53.34" size="1.778" layer="96" rot="R270"/>
 </instance>
-<instance part="Y1" gate="G$1" x="215.9" y="91.44" smashed="yes">
-<attribute name="NAME" x="222.25" y="91.44" size="1.778" layer="95"/>
-</instance>
-<instance part="GND19" gate="1" x="213.36" y="83.82" smashed="yes">
-<attribute name="VALUE" x="210.82" y="81.28" size="1.778" layer="96"/>
-</instance>
-<instance part="GND21" gate="1" x="218.44" y="83.82" smashed="yes">
-<attribute name="VALUE" x="215.9" y="81.28" size="1.778" layer="96"/>
-</instance>
 <instance part="I2C" gate="J1" x="116.84" y="30.48" smashed="yes">
 <attribute name="VALUE" x="111.76" y="25.146" size="1.778" layer="96" font="vector" align="top-left"/>
 <attribute name="NAME" x="111.76" y="38.354" size="1.778" layer="95" font="vector"/>
+</instance>
+<instance part="Y2" gate="G$1" x="220.98" y="93.98" smashed="yes" rot="R90">
+<attribute name="NAME" x="223.52" y="97.79" size="1.778" layer="95"/>
+</instance>
+<instance part="C20" gate="G$1" x="215.9" y="83.82" smashed="yes">
+<attribute name="NAME" x="217.424" y="85.471" size="1.778" layer="95" font="vector"/>
+</instance>
+<instance part="C22" gate="G$1" x="215.9" y="104.14" smashed="yes">
+<attribute name="NAME" x="217.424" y="105.791" size="1.778" layer="95" font="vector"/>
+</instance>
+<instance part="GND19" gate="1" x="226.06" y="86.36" smashed="yes">
+<attribute name="VALUE" x="223.52" y="83.82" size="1.778" layer="96"/>
+</instance>
+<instance part="GND21" gate="1" x="215.9" y="78.74" smashed="yes">
+<attribute name="VALUE" x="213.36" y="76.2" size="1.778" layer="96"/>
+</instance>
+<instance part="GND23" gate="1" x="215.9" y="109.22" smashed="yes" rot="R180">
+<attribute name="VALUE" x="218.44" y="111.76" size="1.778" layer="96" rot="R180"/>
 </instance>
 </instances>
@@
 </segment>
 <segment>
-<pinref part="Y1" gate="G$1" pin="2"/>
-<pinref part="GND19" gate="1" pin="GND"/>
-<wire x1="213.36" y1="86.36" x2="213.36" y2="88.9" width="0.1524" layer="91"/>
-</segment>
-<segment>
-<pinref part="Y1" gate="G$1" pin="4"/>
-<pinref part="GND21" gate="1" pin="GND"/>
-<wire x1="218.44" y1="86.36" x2="218.44" y2="88.9" width="0.1524" layer="91"/>
-</segment>
-<segment>
 <pinref part="I2C" gate="J1" pin="GND"/>
 <wire x1="124.46" y1="27.94" x2="132.08" y2="27.94" width="0.1524" layer="91"/>
 <label x="127" y="27.94" size="1.778" layer="95"/>
+</segment>
+<segment>
+<pinref part="Y2" gate="G$1" pin="4"/>
+<wire x1="223.52" y1="96.52" x2="226.06" y2="96.52" width="0.1524" layer="91"/>
+<wire x1="226.06" y1="96.52" x2="226.06" y2="91.44" width="0.1524" layer="91"/>
+<pinref part="Y2" gate="G$1" pin="2"/>
+<wire x1="226.06" y1="91.44" x2="223.52" y2="91.44" width="0.1524" layer="91"/>
+<wire x1="226.06" y1="91.44" x2="226.06" y2="88.9" width="0.1524" layer="91"/>
+<junction x="226.06" y="91.44"/>
+<pinref part="GND19" gate="1" pin="GND"/>
 </segment>
 </net>
@@
 </segment>
 </net>
-<net name="X48M_P" class="0">
-<segment>
-<pinref part="Y1" gate="G$1" pin="1"/>
+<net name="N$1" class="0">
+<segment>
+<pinref part="Y2" gate="G$1" pin="1"/>
+<wire x1="220.98" y1="91.44" x2="220.98" y2="88.9" width="0.1524" layer="91"/>
+<wire x1="220.98" y1="88.9" x2="215.9" y2="88.9" width="0.1524" layer="91"/>
+<wire x1="215.9" y1="88.9" x2="213.36" y2="88.9" width="0.1524" layer="91"/>
+<wire x1="213.36" y1="88.9" x2="213.36" y2="91.44" width="0.1524" layer="91"/>
 <pinref part="U1" gate="G$1" pin="X48N-P"/>
-<wire x1="200.66" y1="91.44" x2="213.36" y2="91.44" width="0.1524" layer="91"/>
-</segment>
-</net>
-<net name="X48M_N" class="0">
-<segment>
-<pinref part="Y1" gate="G$1" pin="3"/>
-<wire x1="220.98" y1="91.44" x2="218.44" y2="91.44" width="0.1524" layer="91"/>
-<wire x1="220.98" y1="91.44" x2="220.98" y2="93.98" width="0.1524" layer="91"/>
+<wire x1="213.36" y1="91.44" x2="200.66" y2="91.44" width="0.1524" layer="91"/>
+<pinref part="C20" gate="G$1" pin="1"/>
+<wire x1="215.9" y1="88.9" x2="215.9" y2="87.63" width="0.1524" layer="91"/>
+<junction x="215.9" y="88.9"/>
+</segment>
+</net>
+<net name="N$4" class="0">
+<segment>
+<pinref part="Y2" gate="G$1" pin="3"/>
+<wire x1="220.98" y1="96.52" x2="220.98" y2="99.06" width="0.1524" layer="91"/>
+<wire x1="220.98" y1="99.06" x2="215.9" y2="99.06" width="0.1524" layer="91"/>
+<wire x1="215.9" y1="99.06" x2="213.36" y2="99.06" width="0.1524" layer="91"/>
+<wire x1="213.36" y1="99.06" x2="213.36" y2="93.98" width="0.1524" layer="91"/>
 <pinref part="U1" gate="G$1" pin="X48M-N"/>
-<wire x1="220.98" y1="93.98" x2="200.66" y2="93.98" width="0.1524" layer="91"/>
-</segment>
-</net>
-<net name="N$12" class="0">
-<segment>
-<wire x1="220.98" y1="82.55" x2="220.98" y2="81.28" width="0.1524" layer="91"/>
-</segment>
-</net>
+<wire x1="213.36" y1="93.98" x2="200.66" y2="93.98" width="0.1524" layer="91"/>
+<pinref part="C22" gate="G$1" pin="2"/>
+<wire x1="215.9" y1="100.33" x2="215.9" y2="99.06" width="0.1524" layer="91"/>
+<junction x="215.9" y="99.06"/>
+</segment>
+</net>
